File: pcb/pv_test_station/pv_test_station.kicad_sch (KiCad schematic)
At the start: 16 parts, among them IC1 CT426-HSN830DR, J1 Connector_Panel, J2 Connector_load, J3 Conncector 5V, J4 qwiic, J5 i2c, J6 GPS, K1 AZ576-1A-12DE, Q1 2N7002

Commit message: finished pcb
Parts:
- removed J1: Connector_Panel, Connector_Phoenix_MSTB:PhoenixContact_MSTBA_2,5_4-G-5,08_1x04_P5.08mm_Horizontal, symbol Connector:Conn_01x04_Socket
- removed J3: Conncector 5V, Connector_PinHeader_2.54mm:PinHeader_1x02_P2.54mm_Vertical, symbol Connector:Conn_01x02_Socket
- added J1: In, digikey-footprints:PHOENIX_1017521, symbol Connector:Conn_01x02_Socket
- added J10: Bat in, Connector_PinHeader_2.54mm:PinHeader_1x02_P2.54mm_Vertical, symbol Connector:Conn_01x02_Socket
- added J2: Out, digikey-footprints:PHOENIX_1017521, symbol Connector:Conn_01x02_Socket
- added J4: FRAM, Connector_PinSocket_2.54mm:PinSocket_1x08_P2.54mm_Vertical, symbol Connector:Conn_01x08_Socket
- added J7: Temp2, Connector_PinHeader_2.54mm:PinHeader_1x04_P2.54mm_Vertical, symbol Connector:Conn_01x04_Socket
- added U1: ~, digikey-footprints:DCDC, symbol New_Library:DC/DC
- C1: footprint Capacitor_SMD:C_0201_0603Metric -> Capacitor_SMD:C_0603_1608Metric
- D1: footprint Resistor_THT:R_Axial_DIN0204_L3.6mm_D1.6mm_P7.62mm_Horizontal -> digikey-footprints:DIODE_BAR6303WE6327HTSA1_INF
- IC1: footprint SOIC127P600X172-8N -> SamacSys_Parts:SOIC127P600X172-8N
- J3: renamed from J2; value Connector_load -> load; footprint Connector_Phoenix_MSTB:PhoenixContact_MSTBA_2,5_2-G-5,08_1x02_P5.08mm_Horizontal -> digikey-footprints:PHOENIX_1017521
- J6: renamed from J5; value i2c -> Temp1
- J9: renamed from J6; footprint Connector_PinHeader_2.54mm:PinHeader_1x05_P2.54mm_Vertical -> Connector_PinSocket_2.54mm:PinSocket_1x05_P2.54mm_Vertical
- R1, R2: footprint Resistor_SMD:R_0201_0603Metric -> Resistor_SMD:R_0603_1608Metric
- renumbered J4 to J5
Connections:
- net - In is gone; now on net GND: R2.2
- net + In: now also J1.1 (Pin_1)
- net + Out: now also J2.1 (Pin_1)
- net +3.3V: now also A1.2 (3V3), C1.2, IC1.8 (VDD), J4.1 (Pin_1), J7.2 (Pin_2)
- net +5V: now also U1.4 (Vo+)
- net GND: now also J1.2 (Pin_2), J2.2 (Pin_2), J4.2 (Pin_2), J7.1 (Pin_1), U1.3 (Vo-)
- net SCL: now also J4.4 (Pin_4), J7.4 (Pin_4)
- net SDA: now also J4.5 (Pin_5), J7.3 (Pin_3)
- net Relais renamed relais
- new net: J10.1 (Pin_1), U1.2 (Vi+)
- new net: J10.2 (Pin_2), U1.1 (Vi-)
Other:
- moved on the sheet: J9

Commit message: fixed some PCB issues (resistor size, GND on top layer)
Parts:
- J6, J7: footprint Connector_PinHeader_2.54mm:PinHeader_1x04_P2.54mm_Vertical -> Connector_PinSocket_2.54mm:PinSocket_1x04_P2.54mm_Vertical
Changed lines of the file:
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@@
 			)
 		)
-		(property "Footprint" "Connector_PinHeader_2.54mm:PinHeader_1x04_P2.54mm_Vertical"
+		(property "Footprint" "Connector_PinSocket_2.54mm:PinSocket_1x04_P2.54mm_Vertical"
 			(at 237.49 100.33 0)
 			(effects
@@
 			)
 		)
-		(property "Footprint" "Connector_PinHeader_2.54mm:PinHeader_1x04_P2.54mm_Vertical"
+		(property "Footprint" "Connector_PinSocket_2.54mm:PinSocket_1x04_P2.54mm_Vertical"
 			(at 237.49 114.3 0)
 			(effects

Commit message: added docker for db
Parts:
- added R3, R4, R5: nc, Resistor_SMD:R_0603_1608Metric, symbol Device:R
- J1: value In -> PV-In
- J2: value Out -> PV-Out
Connections:
- net +3.3V: now also R3.2, R4.2, R5.2
- net WP: now reaches A1.21 (D9)
- net WP: now also J4.3 (Pin_3)
- net at J4.6 (Pin_6): now also R3.1
- net at J4.7 (Pin_7): now also R4.1
- net at J4.8 (Pin_8): now also R5.1
